File: _saved_STM32F401CCT6.sch (KiCad schematic (older format))
At the start: 37 parts, among them J1 USB_OTG, J2 Conn_02x03_Odd_Even, J3 Conn_01x20_des, J4 Conn_01x05_desc, J5 Conn_01x20, SW1 SW_Push, U1 MIC5219-3.3, U2 STM32F401CCT6, U3 USBLC6-2SC6, Y1 32.786K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

Commit message: Assosciated schematic to footprint
Parts:
- C1, C10, C11, C12, C13, C14, C2, C3, C6, C7, C8, C9: footprint (none) -> Capacitors_SMD:C_0603_HandSoldering
- C4: value C -> 106,0603
- C5: value C -> 104,0603
- D1, D2: footprint (none) -> LEDs:LED_0603_HandSoldering
- J2: footprint (none) -> Pin_Headers:Pin_Header_Straight_2x03_Pitch2.54mm_SMD
- J3, J5: footprint (none) -> Pin_Headers:Pin_Header_Straight_1x20_Pitch2.54mm
- J4: footprint (none) -> Pin_Headers:Pin_Header_Straight_1x05_Pitch2.54mm
- R1, R10, R2, R3, R4, R5, R6, R7, R8, R9: footprint (none) -> Resistors_SMD:R_0603_HandSoldering
- U1: footprint TO_SOT_Packages_SMD:SOT-23-5 -> TO_SOT_Packages_SMD:SOT-23-5_HandSoldering
- U2: footprint (none) -> UFQFPN48:UFQFPN48
- U3: footprint (none) -> TO_SOT_Packages_SMD:SOT-23-6_Handsoldering
