File: _saved_STM32F401CCT6.sch (KiCad schematic (older format))
At the start: 37 parts, among them J1 USB_OTG, J2 Conn_02x03_Odd_Even, J3 Conn_01x20_des, J4 Conn_01x05_desc, J5 Conn_01x20, SW1 SW_Push, U1 MIC5219-3.3, U2 STM32F401CCT6, U3 USBLC6-2SC6, Y1 32.786K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

Commit message: routing
Parts:
- J2: footprint Pin_Headers:Pin_Header_Straight_2x03_Pitch2.54mm_SMD -> Pin_Headers:Pin_Header_Straight_2x03_Pitch2.54mm
Changed lines of the file:
@@
 F 0 "J2" H 2750 1400 50  0000 C CNN
 F 1 "Conn_02x03_Odd_Even" H 2750 1000 50  0000 C CNN
-F 2 "Pin_Headers:Pin_Header_Straight_2x03_Pitch2.54mm_SMD" H 2700 1200 50  0001 C CNN
+F 2 "Pin_Headers:Pin_Header_Straight_2x03_Pitch2.54mm" H 2700 1200 50  0001 C CNN
 F 3 "" H 2700 1200 50  0001 C CNN
 	1    2700 1200

Commit message: routing
Parts:
- J1: footprint Connectors_USB:USB_Micro-B_Molex_47346-0001 -> Connectors_USB:USB_Micro-B_Molex-105017-0001
- Y2: footprint Crystals:Crystal_HC49-U_Vertical -> Crystals:Crystal_HC49-4H_Vertical
Connections:
- net VCC3v3 is gone; now on net VCC: J3.18 (Pin_18), J5.1 (Pin_1), U2.24 (VDD_2), U2.36 (VDD_2), U2.48 (VDD_3), U2.9 (VDDA/VREF+)
- net D-: now reaches J1.2 (D-), R3.2
- net D+: now reaches J1.3 (D+), R4.2
- net ID: now reaches J1.4 (ID), R9.2
Changed lines of the file:
@@
 GND
 Text Label 4600 4400 0    60   ~ 0
-VCC3v3
+VCC
 Text Label 4600 4500 0    60   ~ 0
 PA0
@@
 GND
 Text Label 6650 5600 1    60   ~ 0
-VCC3v3
+VCC
 Text Label 7600 4700 2    60   ~ 0
 PB12
@@
 GND
 Text Label 7600 3600 2    60   ~ 0
-VCC3v3
+VCC
 Text Label 6650 2650 3    60   ~ 0
 SWDCLK
@@
 GND
 Text Label 5550 2650 3    60   ~ 0
-VCC3v3
+VCC
 $Comp
 L STM32F401CCT6 U2
@@
 F 0 "J1" H 700 6750 50  0000 L CNN
 F 1 "USB_OTG" H 700 6650 50  0000 L CNN
-F 2 "Connectors_USB:USB_Micro-B_Molex_47346-0001" H 1050 6250 50  0001 C CNN
+F 2 "Connectors_USB:USB_Micro-B_Molex-105017-0001" H 1050 6250 50  0001 C CNN
 F 3 "" H 1050 6250 50  0001 C CNN
 	1    900  6300
@@
 F 0 "Y2" V 4750 6900 50  0000 C CNN
 F 1 "8MHz" V 4650 6950 50  0000 C CNN
-F 2 "Crystals:Crystal_HC49-U_Vertical" H 4750 6750 50  0001 C CNN
+F 2 "Crystals:Crystal_HC49-4H_Vertical" H 4750 6750 50  0001 C CNN
 F 3 "" H 4750 6750 50  0001 C CNN
 	1    4750 6750
@@
 RESET
 Text Label 4000 4300 2    60   ~ 0
-VCC3v3
+VCC
 Text Label 4000 4400 2    60   ~ 0
 GND
@@
 $EndComp
 Text Label 8300 2750 0    60   ~ 0
-VCC3v3
+VCC
 Text Label 8300 2850 0    60   ~ 0
 GND
@@
 	-1   0    0    1
 $EndComp
+Text Label 1350 6300 0    60   ~ 0
+D-
+Text Label 1350 6400 0    60   ~ 0
+D+
+Text Label 1250 6500 0    60   ~ 0
+ID
 $EndSCHEMATC
