File: _autosave-_autosave-STM32F401CCT6.kicad_pcb (KiCad board)
At the start: 2 copper layers, 37 parts, among them J1 USB_OTG, J2 Conn_02x03_Odd_Even, J3 Conn_01x20_des, J4 Conn_01x05_desc, J5 Conn_01x20, SW1 SW_Push, U1 MIC5219-3.3, U2 STM32F401CCT6, U3 USBLC6-2SC6, Y1 32.786K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

Commit message: routing
Parts:
- J2: footprint Pin_Headers:Pin_Header_Straight_2x03_Pitch2.54mm -> Pin_Headers:Pin_Header_Straight_2x03_Pitch2.54mm_SMD
- moved J2 2.42 mm to (85.8, 104.9), turned to 90 degrees
Routing:
- net (no net): track 1.39 -> 0.00 mm
- net +5V: track 0.00 -> 1.14 mm
- net Net-(J2-Pad3): track 0.00 -> 1.07 mm
